File: hardware/proj/perspection/perspection-v1.sch (EAGLE design)
At the start: 114 parts, among them J1 MICRO-USB-10118192-0001LF, Q1 CSD18533Q5A, Q2 CSD18533Q5A, Q3 CSD18533Q5A, Q4 CSD18533Q5A, Q5 CSD18533Q5A, Q6 CSD18533Q5A, U1 ATUM, U10 DRV8301DCAR, U2 FT232RQ, U3 TPS79933DDCR, U4 MCP73831T-2ACI/OT, U5 TMS320F28069MPZT, U6 DRV8801PWPR, U7 DRV8801PWPR, U8 DRV8801PWPR, U9 DRV8801PWPR

Commit message: changed power LED
Other:
- note added: "i thought the buck converter could only drop to 3.5 also, i think i want 5v to power the LED"
Changed lines of the file:
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@@
 <setting verticaltext="up"/>
 </settings>
-<grid distance="0.1" unitdist="inch" unit="inch" style="lines" multiple="1" display="yes" altdistance="0.01" altunitdist="inch" altunit="inch"/>
+<grid distance="0.1" unitdist="inch" unit="inch" style="lines" multiple="1" display="no" altdistance="0.01" altunitdist="inch" altunit="inch"/>
 <layers>
 <layer number="1" name="Top" color="4" fill="1" visible="no" active="no"/>
@@
 <sheet>
 <plain>
+<text x="149.86" y="114.3" size="1.778" layer="97">i thought the buck converter could only drop to 3.5
+also, i think i want 5v to power the LED</text>
 </plain>
 <instances>
@@
 </schematic>
 </drawing>
+<compatibility>
+<note version="6.3" minversion="6.2.2" severity="warning">
+Since Version 6.2.2 text objects can contain more than one line,
+which will not be processed correctly with this version.
+</note>
+</compatibility>
 </eagle>

Commit message: finished piccolo stuff, for the most part
Parts:
- added C52, C57: 2.2uF, perspection:C0805
- added C53, C54, C55, C56, C58, C59, C60, C61, C62, C80, C81: 0.1uF, perspection:C0402
- added C63, C64, C65: 2200pF, perspection:C0402
- added C66, C67, C68, C69, C70, C71, C72, C73, C74, C75, C76, C77, C78, C79: 2.2uF, perspection:C0402
- added L3: BLM15PD600SN1D, perspection:L0402
- added L4: BKP1005HS221-T, perspection:L0402
- added R40, R41, R42, R43, R44, R45, R46, R47, R48, R49, R50, R51, R52, R53, R54, R55, R56, R57, R58, R59, R60: 0, perspection:R0402
- added R61, R64, R65, R66: 10k, perspection:R0402
- added R62, R63: 1k, perspection:R0402
- added R67, R69, R71, R73: 34.8k, perspection:R0402
- added R68, R70, R72, R74: 4.99k, perspection:R0402
- added R75, R76, R77: 56, perspection:R0402
- added R78: 2.2k, perspection:R0402
- added S1: TACTILE-SWITCH-SMD, perspection:TACTILE-SWITCH-SMD
- added U11: OPA2374AIDCNR, perspection:OPA2374AIDCNR
- C1, C10, C11, C12, C13, C14, C15, C16, C17, C18, C19, C23, C24, C25, C28, C29, C3, C30, C31, C33, C35, C36, C4, C41, C43, C44, C46, C47, C49, C5, C50, C51: device perspection:C0603 -> perspection:C0402
- C37, C38: value 0.1uF -> 1uF
- L1: value FB -> MI0603K300R-10; DIST_NAME (none) -> Digi-key; DIST_PN (none) -> 240-2373-1-ND; MFG_NAME (none) -> Laird-Signal Integrity Products; MFG_PN (none) -> MI0603K300R-10
- R1, R10, R11, R13, R14, R15, R17, R18, R2, R20, R21, R23, R24, R25, R26, R28, R29, R3, R31, R32, R33, R34, R35, R36, R37, R38, R39, R4, R5, R7, R8, R9: device perspection:R0603 -> perspection:R0402
Connections:
- new net !PICCOLO_RESET: C81.1, R78.1, S1.3, S1.4, U5.1.!XRS
- new net !PICCOLO_TRST: U5.1.!TRST
- new net DC_V_FB: C62.1, R43.2, R73.1, R74.2
- new net IC_FB: C65.1, R49.2, R77.2
- new net N$51: C72.1, C73.1, C74.1, C75.1, C76.1, C77.1, L3.2, U5.1.VDDIO
- new net N$56: C78.1, L4.2, U5.1.VDDA
- new net N$58: C66.1, C67.1, C68.1, C69.1, C70.1, C71.1, U5.1.VDD
- new net N$77: R61.1, U11.2.-IN, U11.2.OUT
- new net N$78: C57.1, R61.2, R63.2, U11.1.+IN
- new net N$79: R62.2, R64.1, U11.1.-IN
- new net N$82: R65.1, R66.2, U11.2.+IN
- new net PICCOLO_TCK: U5.1.TCK/GPIO38/XCLK_I
- new net PICCOLO_TDI: U5.1.TDI/GPIO35
- new net PICCOLO_TDO: U5.1.TDO/GPIO37
- new net PICCOLO_TMS: U5.1.TMS/GPIO36
- new net VA_FB: C59.1, R44.2, R67.2, R68.2
- new net VB_FB: C60.1, R45.2, R69.2, R70.2
- new net VC_FB: C61.1, R46.2, R71.2, R72.2
- new net _!DRV_CS: R56.1, U5.2.GPIO27/HRCAP2/EQEP2S/!SPISTEB!/USB0DM
- new net _!FAULT: R40.2, U5.2.GPIO15/ECAP2/SCI_RXDB/!SPISTEB
- new net _!OCTW: R42.1, U5.2.GPIO58/MCLKRA/SCI_TXDB/EPWM7A
- new net _DC_CAL: R60.1, U5.2.GPIO53/EQEP1I/MFSXA
- new net _DC_V_FB: R43.1, U5.1.ADC_INB7
- new net _DRV_SCK: R41.2, U5.2.GPIO14/!TZ3!/SCITXDB/SPICLKB
- new net _DRV_SDI: R57.2, U5.2.GPIO24/ECAP1/EQEP2A/SPISIMOB
- new net _DRV_SDO: R58.2, U5.2.GPIO25/ECAP2/EQEP2B/SPISOMIB
- new net _EN_GATE: R59.1, U5.2.GPIO52/EQEP1S/MCLKXA/!TZ3
- new net _IA_FB: R75.1, U10.CORE.SO1
- new net _IB_FB: R76.1, U10.CORE.SO2
- new net _IC_FB: R64.2, R77.1, U11.1.OUT
- new net _PWM_AH: R50.2, U5.2.GPIO6/EPWM4A/EPWMSYNCI/EPWMSYNCO
- new net _PWM_AL: R51.2, U5.2.GPIO7/EPWM4B/SCIRXDA/ECAP2
- new net _PWM_BH: R52.2, U5.2.GPIO8/EPWM5A/!ADCSOCAO
- new net _PWM_BL: R53.2, U5.2.GPIO9/EPWM5B/SCI_TXDB/ECAP3
- new net _PWM_CH: R54.2, U5.2.GPIO10/EPWM6A/!ADCSOCBO
- new net _PWM_CL: R55.2, U5.2.GPIO11/EPWM6B/SCI_RXDB/ECAP1
- new net _VA_FB: R44.1, U5.1.ADC_INB4/COMP2B/AIO12
- new net _VB_FB: R45.1, U5.1.ADC_INA5
- new net _VC_FB: R46.1, U5.1.ADC_INB5
- new net __IA_FB: R47.1, U5.1.ADC_INA3
- new net __IB_FB: R48.1, U5.1.ADC_INB3
- new net __IC_FB: R49.1, U5.1.ADC_INA4/COMP2A/AIO4
- net !DRV_CS: now also R56.2
- net !FAULT: now also R40.1
- net !OCTW: now also R42.2
- net +12V: now also C52.1, C53.1, R73.2
- net +3V3: now also C56.1, C58.1, C79.1, C80.1, L3.1, L4.1, R65.2, R78.2, U11.1.V+, U5.1.VDD_3VFL
- net +5V: now also C54.1
- net C_ISENSE_N: now also R63.1
- net C_ISENSE_P: now also R62.1
- net DC_CAL: now also R60.2
- net DRV_SCK: now also R41.1
- net DRV_SDI: now also R57.1
- net DRV_SDO: now also R58.1
- net EN_GATE: now also R59.2
- net GND: now also C52.2, C53.2, C54.2, C55.2, C56.2, C57.2, C58.2, C59.2, C60.2, C61.2, C62.2, C63.2, C64.2, C65.2, C66.2, C67.2, C68.2, C69.2, C70.2, C71.2, C72.2, C73.2, C74.2, C75.2, C76.2, C77.2, C78.2, C79.2, C80.2, C81.2, R66.1, R68.1, R70.1, R72.1, R74.1, S1.1, S1.2, U11.1.V-, U5.1.!VREGENZ, U5.1.VREFLO, U5.1.VSS, U5.1.VSSA
- net IA_FB: now also C63.1, R47.2, R75.2; no longer U10.CORE.SO1
- net IB_FB: now also C64.1, R48.2, R76.2; no longer U10.CORE.SO2
- net PWM_AH: now also R50.1
- net PWM_AL: now also R51.1
- net PWM_BH: now also R52.1
- net PWM_BL: now also R53.1
- net PWM_CH: now also R54.1
- net PWM_CL: now also R55.1
- net SH_A: now also R67.1
- net SH_B: now also R69.1
- net SH_C: now also R71.1
- net VBAT: now also C55.1
Other:
- note removed: "i thought the buck converter could only drop to 3.5 also, i think i want 5v to power the LED"

Commit message: parts and LED circuit and shit
Parts:
- added D6: LED-PWR-XLAMP_MX3, perspection:LED-PWR-XLAMP_MX3
- added Q7: NMOS-CSD18533Q5A, perspection:NMOS-CSD18533Q5A
- added R79: (no value), perspection:R0805
- added R80: (no value), perspection:R0402
Connections:
- new net N$59: D6.CATHODE, Q7.D
- new net N$60: Q7.S, R79.2
- new net N$61: Q7.G, R80.1
- net GND: now also R79.1
- net VBAT: now also D6.ANODE
Changed lines of the file:
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@@
 <setting verticaltext="up"/>
 </settings>
-<grid distance="0.1" unitdist="inch" unit="inch" style="lines" multiple="1" display="yes" altdistance="0.01" altunitdist="inch" altunit="inch"/>
+<grid distance="0.1" unitdist="inch" unit="inch" style="lines" multiple="1" display="no" altdistance="0.01" altunitdist="inch" altunit="inch"/>
 <layers>
 <layer number="1" name="Top" color="4" fill="1" visible="no" active="no"/>
@@
 <part name="+3V18" library="perspection" deviceset="+3V3" device=""/>
 <part name="GND63" library="perspection" deviceset="GND" device=""/>
+<part name="P+15" library="perspection" deviceset="VBAT" device=""/>
+<part name="FRAME7" library="perspection" deviceset="A3L-LOC" device=""/>
+<part name="Q7" library="perspection" deviceset="NMOS" device="-CSD18533Q5A"/>
+<part name="D6" library="perspection" deviceset="LED-PWR" device="-XLAMP_MX3"/>
+<part name="R79" library="perspection" deviceset="R" device="0805"/>
+<part name="GND64" library="perspection" deviceset="GND" device=""/>
+<part name="R80" library="perspection" deviceset="R" device="0402"/>
 </parts>
 <sheets>
@@
 </segment>
 </net>
+</nets>
+</sheet>
+<sheet>
+<plain>
+</plain>
+<instances>
+<instance part="P+15" gate="G$1" x="66.04" y="101.6"/>
+<instance part="FRAME7" gate="G$1" x="0" y="0"/>
+<instance part="Q7" gate="G$1" x="63.5" y="83.82"/>
+<instance part="D6" gate="G$1" x="66.04" y="93.98" rot="R270"/>
+<instance part="R79" gate="G$1" x="66.04" y="63.5" rot="R90"/>
+<instance part="GND64" gate="1" x="66.04" y="50.8"/>
+<instance part="R80" gate="G$1" x="53.34" y="81.28" rot="R180"/>
+</instances>
+<busses>
+</busses>
+<nets>
+<net name="VBAT" class="0">
+<segment>
+<pinref part="D6" gate="G$1" pin="ANODE"/>
+<pinref part="P+15" gate="G$1" pin="VBAT"/>
+<wire x1="66.04" y1="99.06" x2="66.04" y2="101.6" width="0.1524" layer="91"/>
+</segment>
+</net>
+<net name="N$59" class="0">
+<segment>
+<pinref part="D6" gate="G$1" pin="CATHODE"/>
+<pinref part="Q7" gate="G$1" pin="D"/>
+<wire x1="66.04" y1="88.9" x2="66.04" y2="91.44" width="0.1524" layer="91"/>
+</segment>
+</net>
+<net name="N$60" class="0">
+<segment>
+<pinref part="Q7" gate="G$1" pin="S"/>
+<pinref part="R79" gate="G$1" pin="2"/>
+<wire x1="66.04" y1="68.58" x2="66.04" y2="78.74" width="0.1524" layer="91"/>
+</segment>
+</net>
+<net name="GND" class="0">
+<segment>
+<pinref part="R79" gate="G$1" pin="1"/>
+<pinref part="GND64" gate="1" pin="GND"/>
+<wire x1="66.04" y1="53.34" x2="66.04" y2="58.42" width="0.1524" layer="91"/>
+</segment>
+</net>
+<net name="N$61" class="0">
+<segment>
+<pinref part="Q7" gate="G$1" pin="G"/>
+<pinref part="R80" gate="G$1" pin="1"/>
+<wire x1="58.42" y1="81.28" x2="60.96" y2="81.28" width="0.1524" layer="91"/>
+</segment>
+</net>

Commit message: started led thing
Parts:
- added R81, R82: (no value), perspection:R0402
- added U12: OPA170AIDBVR, perspection:OPA170AIDBVR
- added VR1: 200k, perspection:R-TRIM-ST4ETA204
Connections:
- new net N$62: R81.2, U12.-IN
- new net N$63: R82.2, VR1.1
- net GND: now also VR1.2
- net N$60: now also R81.1
Changed lines of the file:
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@@
 <part name="GND64" library="perspection" deviceset="GND" device=""/>
 <part name="R80" library="perspection" deviceset="R" device="0402"/>
+<part name="U12" library="perspection" deviceset="OPA170" device="AIDBVR"/>
+<part name="R81" library="perspection" deviceset="R" device="0402"/>
+<part name="R82" library="perspection" deviceset="R" device="0402"/>
+<part name="VR1" library="perspection" deviceset="R-TRIM" device="-ST4ETA204" value="200k"/>
+<part name="GND65" library="perspection" deviceset="GND" device=""/>
 </parts>
 <sheets>
@@
 <instance part="GND64" gate="1" x="66.04" y="50.8"/>
 <instance part="R80" gate="G$1" x="53.34" y="81.28" rot="R180"/>
+<instance part="U12" gate="G$1" x="43.18" y="68.58" rot="R180"/>
+<instance part="R81" gate="G$1" x="58.42" y="71.12" rot="R180"/>
+<instance part="R82" gate="G$1" x="55.88" y="55.88" rot="R270"/>
+<instance part="VR1" gate="G$1" x="55.88" y="43.18" rot="R270"/>
+<instance part="GND65" gate="1" x="55.88" y="30.48"/>
 </instances>
 <busses>
@@
 </segment>
 </net>
-<net name="N$60" class="0">
-<segment>
-<pinref part="Q7" gate="G$1" pin="S"/>
-<pinref part="R79" gate="G$1" pin="2"/>
-<wire x1="66.04" y1="68.58" x2="66.04" y2="78.74" width="0.1524" layer="91"/>
-</segment>
-</net>
 <net name="GND" class="0">
 <segment>
@@
 <wire x1="66.04" y1="53.34" x2="66.04" y2="58.42" width="0.1524" layer="91"/>
 </segment>
+<segment>
+<pinref part="VR1" gate="G$1" pin="2"/>
+<pinref part="GND65" gate="1" pin="GND"/>
+<wire x1="55.88" y1="33.02" x2="55.88" y2="38.1" width="0.1524" layer="91"/>
+</segment>
 </net>
 <net name="N$61" class="0">
@@
 </segment>
 </net>
+<net name="N$62" class="0">
+<segment>
+<pinref part="R81" gate="G$1" pin="2"/>
+<pinref part="U12" gate="G$1" pin="-IN"/>
+<wire x1="50.8" y1="71.12" x2="53.34" y2="71.12" width="0.1524" layer="91"/>
+</segment>
+</net>
+<net name="N$60" class="0">
+<segment>
+<pinref part="Q7" gate="G$1" pin="S"/>
+<pinref part="R79" gate="G$1" pin="2"/>
+<wire x1="66.04" y1="78.74" x2="66.04" y2="71.12" width="0.1524" layer="91"/>
+<pinref part="R81" gate="G$1" pin="1"/>
+<wire x1="66.04" y1="71.12" x2="66.04" y2="68.58" width="0.1524" layer="91"/>
+<wire x1="63.5" y1="71.12" x2="66.04" y2="71.12" width="0.1524" layer="91"/>
+<junction x="66.04" y="71.12"/>
+</segment>
+</net>
+<net name="N$63" class="0">
+<segment>
+<pinref part="R82" gate="G$1" pin="2"/>
+<pinref part="VR1" gate="G$1" pin="1"/>
+<wire x1="55.88" y1="48.26" x2="55.88" y2="50.8" width="0.1524" layer="91"/>
+</segment>
+</net>

Commit message: i dont fuckin kno what i did
Parts:
- added C82, C83, C84, C85, C86, C87: 220uF, perspection:CPOL-PANASONIC-6.3MM-SMD-220UF-25V
- added C88, C89, C90, C93: 0.1uF, perspection:C0402
- added C91, C92: 12.5pF, perspection:C0402
- added J2: 1X6-PTSA_1.5/6-3.5-Z, perspection:1X6-PTSA_1.5/6-3.5-Z
- added J3: 1X2-PTSA_1.5/2-3.5-Z, perspection:1X2-PTSA_1.5/2-3.5-Z
- added J4, J5: 1X2-JST-PH-SMD, perspection:1X2-JST-PH-SMD
- added Q10: NMOS-CSD18533Q5A, perspection:NMOS-CSD18533Q5A
- added Q11: IRFML8244TRPBF, perspection:IRFML8244TRPBF
- added Q8, Q9: BSS138L, perspection:BSS138L
- added R83, R84, R85, R86: 10k, perspection:R0603
- added R87, R88: 4.7k, perspection:R0603
- added R89: 1k, perspection:R0402
- added R90: 100, perspection:R0402
- added R91: DNP, perspection:R0402
- added R92: DNP, perspection:R0805
- added S2: SSA22/DPDT, perspection:SSA22/DPDT
- added U13: BNO055, perspection:BNO055
- added Y1: 32.768kHz, perspection:CM200C32768HZFT
- Q1, Q2, Q3, Q4, Q5, Q6: value CSD18533Q5A -> NMOS-CSD18533Q5A; device perspection:CSD18533Q5A -> perspection:NMOS-CSD18533Q5A
- R80: value (none) -> 10
- R81: value (none) -> 0
Connections:
- new net LED_PWM: Q8.G
- new net N$64: J2.1, U6.OUT+
- new net N$65: J2.2, U6.OUT-
- new net N$66: J2.3, U7.OUT+
- new net N$67: J2.4, U7.OUT-
- new net N$68: J2.5, U8.OUT+
- new net N$69: J2.6, U8.OUT-
- new net N$70: J3.1, U9.OUT+
- new net N$71: J3.2, U9.OUT-
- new net N$72: R84.2, U13.PS1
- new net N$73: R83.2, U13.PS0
- new net N$74: C92.1, U13.XIN32, Y1.3
- new net N$75: C88.2, U13.CAP
- new net N$76: C91.1, U13.XOUT32, Y1.1
- new net N$80: R85.2, U13.COM3
- new net N$81: Q9.D, R89.1, U3.EN
- new net N$83: Q8.D, U12.+IN, VR1.WIPER
- new net N$84: R80.2, U12.OUT
- new net N$85: R86.1, U13.!BOOT_LOAD_PIN
- new net N$86: J5.2, Q10.D, R92.1
- new net N$87: Q9.G, R90.1
- new net N$88: J4.2, Q11.D, R91.1
- net !ATUM_RESET: now also S2.1.1
- net !DTR_FTDI: now also S2.2.2
- net !RTS_FTDI: now also S2.1.2
- net +12V: now also C82.+, C83.+, C84.+, C85.+, C86.+, C87.+, C93.1, D6.ANODE, J5.1, Q10.G, R90.2, U12.V+
- net +3V3: now also C89.1, C90.1, R82.1, R86.2, R87.2, R88.2, U13.!RESET, U13.VDD, U13.VDDIO
- net BOOTLOADER_CTRL: now also S2.2.1
- net GND: now also C82.-, C83.-, C84.-, C85.-, C86.-, C87.-, C88.1, C89.2, C90.2, C91.2, C92.2, C93.2, Q10.S, Q11.S, Q8.S, Q9.S, R83.1, R84.1, R85.1, R91.2, R92.2, U12.V-, U13.COM2, U13.GND, U13.GNDIO, Y1.2
- net I2C_SCL: now also R88.1, U13.COM1
- net I2C_SDA: now also R87.1, U13.COM0
- net VBAT: now also J4.1, Q11.G, R89.2; no longer D6.ANODE, U3.EN
Other:
- moved on the sheet: C1, C10, C11, C12, C13, C14, C15, C16, C17, C18, C19, C2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

Commit message: finished them dots
Parts:
- added C94: 22uF, perspection:C1206
- added J6, J7: JTAG-ARM_TC-10, perspection:JTAG-ARM_TC-10
- added L5: BLM15PD600SN1D, perspection:L0402
- J5: value 1X2-JST-PH-SMD -> 1X2-0428202213; device perspection:1X2-JST-PH-SMD -> perspection:1X2-0428202213
Connections:
- removed net !PICCOLO_TRST: U5.1.!TRST
- removed net ATUM_B6: U1.B6
- removed net PICCOLO_TCK: U5.1.TCK/GPIO38/XCLK_I
- removed net PICCOLO_TDI: U5.1.TDI/GPIO35
- removed net PICCOLO_TDO: U5.1.TDO/GPIO37
- removed net PICCOLO_TMS: U5.1.TMS/GPIO36
- new net N$89: C94.1, L5.2, U1.VCC
- new net N$90: J6.TDI, U1.B6
- new net N$91: J7.TMS, U5.1.TMS/GPIO36
- new net N$92: J7.TCK, U5.1.TCK/GPIO38/XCLK_I
- new net N$93: J7.TDI, U5.1.TDI/GPIO35
- new net N$94: J7.TDO, U5.1.TDO/GPIO37
- new net N$95: J7.RESET, U5.1.!TRST
- net !ATUM_RESET: now also J6.RESET
- net +3V3: now also J6.VCC, L5.1; no longer U1.VCC
- net ATUM_TCK: now also J6.TCK
- net ATUM_TDO: now also J6.TDO
- net ATUM_TMS: now also J6.TMS
- net GND: now also C94.2, J6.GND, J7.GND
- net N$51: now also J7.VCC
Other:
- moved on the sheet: C66, C67, C68, C69, C70, C71, C72, C73, C74, C75, C76, C77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

Commit message: boz is making me commit
Parts:
- added J8: 1X3-0.1IN_THRUHOLE, perspection:1X3-0.1IN_THRUHOLE
- C20, C21, C22, C26, C37, C38, C6: device perspection:C0603 -> perspection:C0402
- C45, C57: device perspection:C0805 -> perspection:C0402
- R22, R27, R30: device perspection:R-SENSE3637-0.01 -> perspection:R-SENSE2010-0.01
- R83, R84, R85, R86, R87, R88: device perspection:R0603 -> perspection:R0402
Connections:
- net N$43 renamed DVDD
- net N$44 renamed AVDD
- net N$46 renamed PH
- net N$47 renamed RT_CLK
- net N$48 renamed BST_BK
- net N$49 renamed DTC
- net N$50 renamed SS_TR
- net N$52 renamed PWRGD
- net N$53 renamed GVDD
- net N$54 renamed _COMP
- net N$55 renamed COMP
- net N$57 renamed VFB
- net N$86 renamed +12V_GND
- net N$88 renamed VBAT_GND
- net GND: now also D6.HEAT
- net SH_A: now also J8.1
- net SH_B: now also J8.2
- net SH_C: now also J8.3
Other:
- moved on the sheet: C31, C34, C35, D6, Q5, Q6, R28, R29, R30, U10.C

Commit message: TAKE THIS SHIT JASON
Parts:
- S1: value TACTILE-SWITCH-SMD -> TACTILE-SWITCH-EVQP2; device perspection:TACTILE-SWITCH-SMD -> perspection:TACTILE-SWITCH-EVQP2
Connections:
- net N$16 renamed SENSE1
- net N$17 renamed _VPROPI1
- net N$21 renamed SENSE2
- net N$25 renamed SENSE3
- net N$26 renamed _VPROPI2
- net N$27 renamed _VPROPI3
- net N$31 renamed AUX_SENSE
- net N$32 renamed _AUX_VPROPI
- net N$64 renamed M1+
- net N$65 renamed M1-
- net N$66 renamed M2+
- net N$67 renamed M2-
- net N$68 renamed M3+
- net N$69 renamed M3-
- net N$70 renamed M_AUX+
- net N$71 renamed M_AUX-
Changed lines of the file:
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@@
 <part name="GND60" library="perspection" deviceset="GND" device=""/>
 <part name="GND61" library="perspection" deviceset="GND" device=""/>
-<part name="S1" library="perspection" deviceset="TACTILE-SWITCH" device="-SMD"/>
+<part name="S1" library="perspection" deviceset="TACTILE-SWITCH" device="-EVQP2" value="TACTILE-SWITCH-EVQP2"/>
 <part name="R78" library="perspection" deviceset="R" device="0402" value="2.2k"/>
 <part name="C81" library="perspection" deviceset="C" device="0402" value="0.1uF"/>
@@
 </segment>
 </net>
-<net name="N$16" class="0">
+<net name="SENSE1" class="0">
 <segment>
 <pinref part="U6" gate="G$1" pin="SENSE"/>
@@
 </segment>
 </net>
-<net name="N$21" class="0">
+<net name="SENSE2" class="0">
 <segment>
 <pinref part="U7" gate="G$1" pin="SENSE"/>
@@
 </segment>
 </net>
-<net name="N$25" class="0">
+<net name="SENSE3" class="0">
 <segment>
 <pinref part="U8" gate="G$1" pin="SENSE"/>
@@
 </segment>
 </net>
-<net name="N$17" class="0">
+<net name="_VPROPI1" class="0">
 <segment>
 <pinref part="U6" gate="G$1" pin="VPROPI"/>
@@
 </segment>
 </net>
-<net name="N$26" class="0">
+<net name="_VPROPI2" class="0">
 <segment>
 <pinref part="U7" gate="G$1" pin="VPROPI"/>
@@
 </segment>
 </net>
-<net name="N$27" class="0">
+<net name="_VPROPI3" class="0">
 <segment>
 <pinref part="R14" gate="G$1" pin="2"/>
@@
 </segment>
 </net>
-<net name="N$31" class="0">
+<net name="AUX_SENSE" class="0">
 <segment>
 <pinref part="U9" gate="G$1" pin="SENSE"/>
@@
 </segment>
 </net>
-<net name="N$32" class="0">
+<net name="_AUX_VPROPI" class="0">
 <segment>
 <pinref part="U9" gate="G$1" pin="VPROPI"/>
@@
 </segment>
 </net>
-<net name="N$64" class="0">
+<net name="M1+" class="0">
 <segment>
 <pinref part="J2" gate="G$1" pin="1"/>
@@
 </segment>
 </net>
-<net name="N$65" class="0">
+<net name="M1-" class="0">
 <segment>
 <pinref part="U6" gate="G$1" pin="OUT-"/>
@@
 </segment>
 </net>
-<net name="N$66" class="0">
+<net name="M2+" class="0">
 <segment>
 <pinref part="J2" gate="G$1" pin="3"/>
@@
 </segment>
 </net>
-<net name="N$67" class="0">
+<net name="M2-" class="0">
 <segment>
 <pinref part="U7" gate="G$1" pin="OUT-"/>
@@
 </segment>
 </net>
-<net name="N$68" class="0">
+<net name="M3+" class="0">
 <segment>
 <pinref part="J2" gate="G$1" pin="5"/>
@@
 </segment>
 </net>
-<net name="N$69" class="0">
+<net name="M3-" class="0">
 <segment>
 <pinref part="U8" gate="G$1" pin="OUT-"/>
@@
 </segment>
 </net>
-<net name="N$70" class="0">
+<net name="M_AUX+" class="0">
 <segment>
 <pinref part="U9" gate="G$1" pin="OUT+"/>
@@
 </segment>
 </net>
-<net name="N$71" class="0">
+<net name="M_AUX-" class="0">
 <segment>
 <pinref part="U9" gate="G$1" pin="OUT-"/>
